File: wolfDemo/wolfDemo_ST33/wolfDemo-STSAFE.kicad_sch (KiCad schematic)
At the start: 12 parts, among them CON1 MIKROBUS_MODULE_CONN, IC1 ST33KTPM2I3WBZA9

Commit message: Update board to 1.2
Also update README
Parts:
- added R2, R7: 1K, Resistor_SMD:R_0603_1608Metric_Pad0.98x0.95mm_HandSolder, symbol Device:R
- added R8, R9: 4.7K, Resistor_SMD:R_0603_1608Metric_Pad0.98x0.95mm_HandSolder, symbol Device:R
- added SW1: SW_SPDT, Button_Switch_SMD:SW_SPDT_PCM12, symbol Switch:SW_SPDT
Connections:
- net +3.3V: now also R2.1, R7.1, R8.1
- net GND: now also R9.2
- net SDA: now reaches CON1.P11 (SDA)
- net SDA: now also IC1.29 (2C_SDA/GPIO_6), R7.2
- net SCL: now reaches CON1.P12 (SCL)
- net SCL: now also IC1.30 (I2C_SCL/GPIO_5), R2.2
- net I2CSEL: now reaches IC1.6 (GPI_I2C_SELECT)
- net I2CSEL: now also SW1.2 (B)
- new net: R8.2, SW1.1 (A)
- new net: R9.1, SW1.3 (C)
Other:
- note added: "GND for I2C, 3.3v for SPI"
