File: wolfDemo/wolfDemo_STM32U585/wolfSTM32-Demo.kicad_pcb (KiCad board)
At the start: 2 copper layers, 111.1 x 135.6 mm, 71 parts, among them J1 Conn_ARM_SWD_TagConnect_TC203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, J2 USB_C_Receptacle_USB2.0_14P, J3 1, J4 2, J5 Conn_ARM_JTAG_SWD_10, Q1 MMBT3904, Q2 MMBT3904, Q3 MMBT3904, Q4 MMBT3904, SW1 SW_Push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

Commit message: Update board to 1.2
Also update README
Parts:
- turned R8 to 90 degrees
